Commit message: angular momentum saturation constraint added in locomotion_nmpc definition

File: crawling_vispa_model/urdf/VISPA_crawling.urdf (robot description, URDF)
Before this commit: robot VISPA, 16 links, 15 joints
Links:
- link Link_0: geometry collision mesh filename=mpc/crawling_vispa_model/meshes/torso.stl; visual mesh filename=mpc/crawling_vispa_model/meshes/torso.stl
- link Link_1_a: geometry collision mesh filename=mpc/crawling_vispa_model/meshes/link1.stl; visual mesh filename=mpc/crawling_vispa_model/meshes/link1.stl
- link Link_1_b: geometry collision mesh filename=mpc/crawling_vispa_model/meshes/link1.stl; visual mesh filename=mpc/crawling_vispa_model/meshes/link1.stl
- link Link_2_a: geometry collision mesh filename=mpc/crawling_vispa_model/meshes/link2_0_5.stl; visual mesh filename=mpc/crawling_vispa_model/meshes/link2_0_5.stl
- link Link_2_b: geometry collision mesh filename=mpc/crawling_vispa_model/meshes/link2_0_5.stl; visual mesh filename=mpc/crawling_vispa_model/meshes/link2_0_5.stl
- link Link_3_a: geometry collision mesh filename=mpc/crawling_vispa_model/meshes/link3.stl; visual mesh filename=mpc/crawling_vispa_model/meshes/link3.stl
- link Link_3_b: geometry collision mesh filename=mpc/crawling_vispa_model/meshes/link3.stl; visual mesh filename=mpc/crawling_vispa_model/meshes/link3.stl
- link Link_4_a: geometry collision mesh filename=mpc/crawling_vispa_model/meshes/link4.stl; visual mesh filename=mpc/crawling_vispa_model/meshes/link4.stl
- link Link_4_b: geometry collision mesh filename=mpc/crawling_vispa_model/meshes/link4.stl; visual mesh filename=mpc/crawling_vispa_model/meshes/link4.stl
- link Link_5_a: geometry collision mesh filename=mpc/crawling_vispa_model/meshes/link5.stl; visual mesh filename=mpc/crawling_vispa_model/meshes/link5.stl
- link Link_5_b: geometry collision mesh filename=mpc/crawling_vispa_model/meshes/link5.stl; visual mesh filename=mpc/crawling_vispa_model/meshes/link5.stl
- link Link_6_a: geometry collision mesh filename=mpc/crawling_vispa_model/meshes/link6.stl; visual mesh filename=mpc/crawling_vispa_model/meshes/link6.stl
- link Link_6_b: geometry collision mesh filename=mpc/crawling_vispa_model/meshes/link6.stl; visual mesh filename=mpc/crawling_vispa_model/meshes/link6.stl
