Commit message: Underactuated Walking case working suboptimal with non-linear saturation constraint in 3D

File: crawling_vispa_model/urdf/vispa2D.urdf (robot description, URDF)
Before this commit: robot VISPA, 16 links, 15 joints
Links:
- link Link_0: mass 50 -> 0.627
Joints:
- joint Joint_1_a: origin xyz=-0.240  0.41469 -0.064498 rpy=-2.0944 0 0.5236 -> xyz=-0.240  0.41469 -0.064498 rpy=0 0 0; type revolute -> fixed
- joint Joint_1_b: origin xyz=-0.240  -0.41469 -0.064498 rpy=1.047197551 3.14149265359 -0.5236 -> xyz=-0.240  -0.41469 -0.064498 rpy=0 0 0 ; type revolute -> fixed
- joint Joint_2_b: axis 0 0 1 -> 0 0 -1
- joint Joint_4_a: type revolute -> fixed
- joint Joint_4_b: type revolute -> fixed
- joint Joint_6_a: type revolute -> fixed
- joint Joint_6_b: type revolute -> fixed

Commit message: added momentum evaluation function

File: crawling_vispa_model/urdf/vispa2D.urdf (robot description, URDF)
Before this commit: robot VISPA, 16 links, 15 joints
Links:
- link Link_0: mass 0.627 -> 70
